Commit message: feat: Fixed robot joints to continous and fixed friction coefficients
The robot works, moves in a straight line and follows an arc if steer is given

TODO: Fix steady state control inputs (free Moving). invert wheel joint axes to make front +ve

File: src/latty_chassis/urdf/latty_model.urdf.xacro (robot description, xacro)
@@ -4,11 +4,13 @@
   <xacro:property name="wheel_radius" value="0.1"/>
   <xacro:property name="wheel_length" value="0.06"/>
+  <xacro:property name="front_wheel_radius" value="0.03"/>
+  <xacro:property name="front_wheel_length" value="0.02"/>
   <xacro:property name="wheelbase" value="0.34"/>
   <!-- Chassis -->
   <link name="chassis">
     <inertial>
-      <origin xyz="0 0 0.1" rpy="0 0 0"/>
-      <mass value="10.0"/>
-      <inertia ixx="0.5" iyy="1.0" izz="0.1" ixy="0" ixz="0" iyz="0"/>
+      <origin xyz="0 0 0.05" rpy="0 0 0"/>
+      <mass value="30.0"/>
+      <inertia ixx="1.25" iyy="4.25" izz="5.0" ixy="0" ixz="0" iyz="0"/>
     </inertial>
     <visual>
@@ -35,5 +37,5 @@
       <origin xyz="0 0 0" rpy="0 0 0"/>
       <geometry>
-        <box size="0.03 0.03 0.04"/>
+        <box size="0.03 0.02 0.04"/>
       </geometry>
     </visual>
@@ -41,13 +43,51 @@
       <origin xyz="0 0 0" rpy="0 0 0"/>
       <geometry>
-        <box size="0.06 0.03 0.06"/>
-      </geometry>
-    </collision>
-  </link>
-  <!-- Wheels -->
+        <box size="0.03 0.02 0.04"/>
+      </geometry>
+    </collision>
+  </link>
+  <!-- Front left wheel -->
+  <link name="front_left_wheel">
+    <inertial>
+      <mass value="1.5"/>
+      <inertia ixx="0.000388" iyy="0.000388" izz="0.000675" ixy="0.0" ixz="0.0" iyz="0.0"/>
+    </inertial>
+    <visual>
+      <origin xyz="0 0 0" rpy="0 1.5707 1.5707"/>
+      <geometry>
+        <cylinder length="${front_wheel_length}" radius="${front_wheel_radius}"/>
+      </geometry>
+    </visual>
+    <collision>
+      <origin xyz="0 0 0" rpy="0 1.5707 1.5707"/>
+      <geometry>
+        <cylinder length="${front_wheel_length}" radius="${front_wheel_radius}"/>
+      </geometry>
+    </collision>
+  </link>
+  <!-- Front right wheel -->
+  <link name="front_right_wheel">
+    <inertial>
+      <mass value="1.5"/>
+      <inertia ixx="0.000388" iyy="0.000388" izz="0.000675" ixy="0.0" ixz="0.0" iyz="0.0"/>
+    </inertial>
+    <visual>
+      <origin xyz="0 0 0" rpy="0 1.5707 1.5707"/>
+      <geometry>
+        <cylinder length="${front_wheel_length}" radius="${front_wheel_radius}"/>
+      </geometry>
+    </visual>
+    <collision>
+      <origin xyz="0 0 0" rpy="0 1.5707 1.5707"/>
+      <geometry>
+        <cylinder length="${front_wheel_length}" radius="${front_wheel_radius}"/>
+      </geometry>
+    </collision>
+  </link>
+  <!-- Rear Wheels -->
   <link name="left_wheel">
     <inertial>
-      <mass value="2.0"/>
-      <inertia ixx="0.0056" iyy="0.0056" izz="0.01" ixy="0.0" ixz="0.0" iyz="0.0"/>
+      <mass value="5.0"/>
+      <inertia ixx="0.0143" iyy="0.0143" izz="0.025" ixy="0.0" ixz="0.0" iyz="0.0"/>
     </inertial>
     <visual>
@@ -66,6 +106,6 @@
   <link name="right_wheel">
     <inertial>
-      <mass value="2.0"/>
-      <inertia ixx="0.0056" iyy="0.0056" izz="0.01" ixy="0.0" ixz="0.0" iyz="0.0"/>
+      <mass value="5.0"/>
+      <inertia ixx="0.0143" iyy="0.0143" izz="0.025" ixy="0.0" ixz="0.0" iyz="0.0"/>
     </inertial>
     <visual>
@@ -88,10 +128,34 @@
   <gazebo reference="left_wheel">
     <material>Gazebo/Black</material>
+    <mu1>1.0</mu1>
+    <mu2>1.0</mu2>
+    <kp>1000000.0</kp>
+    <kd>1.0</kd>
   </gazebo>
   <gazebo reference="right_wheel">
     <material>Gazebo/Black</material>
+    <mu1>1.0</mu1>
+    <mu2>1.0</mu2>
+    <kp>1000000.0</kp>
+    <kd>1.0</kd>
   </gazebo>
   <gazebo reference="steer_knuckle">
     <material>Gazebo/Grey</material>
+    <mu1>0.1</mu1>    <!-- Low friction coefficient -->
+    <mu2>0.1</mu2>    <!-- Low friction coefficient -->
+  </gazebo>
+  <gazebo reference="front_left_wheel">
+    <material>Gazebo/Black</material>
+    <mu1>1.0</mu1>
+    <mu2>1.0</mu2>
+    <kp>1000000.0</kp>
+    <kd>1.0</kd>
+  </gazebo>
+  <gazebo reference="front_right_wheel">
+    <material>Gazebo/Black</material>
+    <mu1>1.0</mu1>
+    <mu2>1.0</mu2>
+    <kp>1000000.0</kp>
+    <kd>1.0</kd>
   </gazebo>
   <!-- Joints -->
@@ -104,19 +168,33 @@
     <dynamics damping="0.5"/>
   </joint>
-  <joint name="left_wheel_joint" type="revolute">
+  <!-- Front wheel joints attached to knuckle -->
+  <joint name="front_left_wheel_joint" type="continuous">
+    <parent link="steer_knuckle"/>
+    <child link="front_left_wheel"/>
+    <origin xyz="0 0.02 -0.015" rpy="0 0 0"/>
+    <axis xyz="0 1 0"/>
+    <dynamics damping="0.1" friction="0.05"/>
+  </joint>
+  <joint name="front_right_wheel_joint" type="continuous">
+    <parent link="steer_knuckle"/>
+    <child link="front_right_wheel"/>
+    <origin xyz="0 -0.02 -0.015" rpy="0 0 0"/>
+    <axis xyz="0 1 0"/>
+    <dynamics damping="0.1" friction="0.05"/>
+  </joint>
+  <!-- Rear wheel joints -->
+  <joint name="left_wheel_joint" type="continuous">
     <parent link="chassis"/>
     <child link="left_wheel"/>
-    <origin xyz="0.1 0.13 ${wheel_radius}" rpy="0 0 0"/>
-    <axis xyz="0 0 1"/>
-    <limit effort="5" velocity="10"/>
-    <dynamics damping="0.1" friction="0.01"/>
-  </joint>
-  <joint name="right_wheel_joint" type="revolute">
+    <origin xyz="0.1 0.13 0.085" rpy="0 0 0"/>
+    <axis xyz="0 1 0"/>
+    <dynamics damping="1.0" friction="0.1"/>
+  </joint>
+  <joint name="right_wheel_joint" type="continuous">
     <parent link="chassis"/>
     <child link="right_wheel"/>
-    <origin xyz="0.1 -0.13 ${wheel_radius}" rpy="0 0 0"/>
-    <axis xyz="0 0 1"/>
-    <limit effort="5" velocity="10"/>
-    <dynamics damping="0.1" friction="0.01"/>
+    <origin xyz="0.1 -0.13 0.085" rpy="0 0 0"/>
+    <axis xyz="0 1 0"/>
+    <dynamics damping="1.0" friction="0.1"/>
   </joint>
   <!-- ros2_control hardware definition -->

Commit message: working manual control node. Ncurses TUI runs on a different thread from ros

File: src/latty_chassis/urdf/latty_model.urdf.xacro (robot description, xacro)
@@ -188,6 +188,6 @@
     <child link="left_wheel"/>
     <origin xyz="0.1 0.13 0.085" rpy="0 0 0"/>
-    <axis xyz="0 1 0"/>
-    <dynamics damping="1.0" friction="0.1"/>
+    <axis xyz="0 -1 0"/>
+    <dynamics damping="5.0" friction="0.5"/>
   </joint>
   <joint name="right_wheel_joint" type="continuous">
@@ -195,6 +195,6 @@
     <child link="right_wheel"/>
     <origin xyz="0.1 -0.13 0.085" rpy="0 0 0"/>
-    <axis xyz="0 1 0"/>
-    <dynamics damping="1.0" friction="0.1"/>
+    <axis xyz="0 -1 0"/>
+    <dynamics damping="5.0" friction="0.5"/>
   </joint>
   <!-- ros2_control hardware definition -->

Commit message: Added rviz params and working joint_states_pos for rviz odom

File: src/latty_chassis/urdf/latty_model.urdf.xacro (robot description, xacro)
@@ -207,10 +207,20 @@
       <state_interface name="position"/>
     </joint>
+    <joint name="front_left_wheel_joint">
+      <state_interface name="position"/>
+      <state_interface name="velocity"/>
+    </joint>
+    <joint name="front_right_wheel_joint">
+      <state_interface name="position"/>
+      <state_interface name="velocity"/>
+    </joint>
     <joint name="left_wheel_joint">
       <command_interface name="velocity"/>
+      <state_interface name="position"/>
       <state_interface name="velocity"/>
     </joint>
     <joint name="right_wheel_joint">
       <command_interface name="velocity"/>
+      <state_interface name="position"/>
       <state_interface name="velocity"/>
     </joint>

Commit message: working odom with correct sign conventions. fixed urdf to point robot front axis along +x. rviz odom working, localisation with little drift over short time.

File: src/latty_chassis/urdf/latty_model.urdf.xacro (robot description, xacro)
@@ -6,5 +6,6 @@
   <xacro:property name="front_wheel_radius" value="0.03"/>
   <xacro:property name="front_wheel_length" value="0.02"/>
-  <xacro:property name="wheelbase" value="0.34"/>
+  <xacro:property name="wheelbase" value="0.25"/>
+  <link name="base_link"/>
   <!-- Chassis -->
   <link name="chassis">
@@ -160,4 +161,10 @@
   </gazebo>
   <!-- Joints -->
+  <joint name="base_to_chassis" type="fixed">
+    <parent link="base_link"/>
+    <child link="chassis"/>
+    <!-- Rotate chassis 180 deg around z if needed -->
+    <origin xyz="0 0 0" rpy="0 0 3.14159"/>
+  </joint>
   <joint name="front_steer_joint" type="revolute">
     <parent link="chassis"/>
@@ -173,5 +180,5 @@
     <child link="front_left_wheel"/>
     <origin xyz="0 0.02 -0.015" rpy="0 0 0"/>
-    <axis xyz="0 1 0"/>
+    <axis xyz="0 -1 0"/>
     <dynamics damping="0.1" friction="0.05"/>
   </joint>
@@ -180,5 +187,5 @@
     <child link="front_right_wheel"/>
     <origin xyz="0 -0.02 -0.015" rpy="0 0 0"/>
-    <axis xyz="0 1 0"/>
+    <axis xyz="0 -1 0"/>
     <dynamics damping="0.1" friction="0.05"/>
   </joint>

Commit message: added imu for localisation. TODO: Move IMU and base_link frame to align with rear_wheel axis

File: src/latty_chassis/urdf/latty_model.urdf.xacro (robot description, xacro)
@@ -123,4 +123,24 @@
     </collision>
   </link>
+  <!-- IMU -->
+  <link name="imu_link">
+    <collision>
+      <origin xyz="0 0 0" rpy="0 0 0"/>
+      <geometry>
+        <box size="0.02 0.02 0.01"/>
+      </geometry>
+    </collision>
+    <inertial>
+      <origin xyz="0 0 0"  rpy="0 0 0"/>
+      <mass value="0.01"/>
+      <inertia ixx="1e-6" iyy="1e-6" izz="1e-6" ixy="0" ixz="0" iyz="0"/>
+    </inertial>
+    <visual>
+      <origin xyz="0 0 0" rpy="0 0 0"/>
+      <geometry>
+        <box size="0.05 0.05 0.02"/>
+      </geometry>
+    </visual>
+  </link>
   <!-- Gazebo material overrides -->
   <gazebo reference="chassis">
@@ -159,4 +179,7 @@
     <kp>1000000.0</kp>
     <kd>1.0</kd>
+  </gazebo>
+  <gazebo reference="imu_link">
+    <material>Gazebo/Grey</material>
   </gazebo>
   <!-- Joints -->
@@ -166,4 +189,9 @@
     <!-- Rotate chassis 180 deg around z if needed -->
     <origin xyz="0 0 0" rpy="0 0 3.14159"/>
+  </joint>
+  <joint name="imu_joint" type="fixed">
+    <parent link="base_link"/>
+    <child link="imu_link"/>
+    <origin xyz="-0.05 0 0.16" rpy="0 0 0"/>
   </joint>
   <joint name="front_steer_joint" type="revolute">
@@ -238,3 +266,17 @@
     </plugin>
   </gazebo>
+  <gazebo reference="imu_link">
+    <sensor name="imu_sensor" type="imu">
+      <always_on>true</always_on>
+      <update_rate>100.0</update_rate>
+      <visualize>true</visualize>
+      <plugin name="imu_plugin" filename="libgazebo_ros_imu_sensor.so">
+        <ros>
+          <namespace>/</namespace>
+          <remappings>~/out:=/imu</remappings>
+        </ros>
+        <frame_name>imu_link</frame_name>
+      </plugin>
+    </sensor>
+  </gazebo>
 </robot>

Commit message: integrating angular velocity to get orientation instead of using imu's orientation

File: src/latty_chassis/urdf/latty_model.urdf.xacro (robot description, xacro)
@@ -261,4 +261,6 @@
     </joint>
   </ros2_control>
+  <xacro:property name="noise" value="1e-3"/>
+  <xacro:property name="drift" value="1e-5"/>
   <gazebo>
     <plugin name="gazebo_ros2_control" filename="libgazebo_ros2_control.so">
@@ -269,6 +271,63 @@
     <sensor name="imu_sensor" type="imu">
       <always_on>true</always_on>
-      <update_rate>100.0</update_rate>
+      <update_rate>100.0</update_rate>   <!-- 100 Hz IMU -->
       <visualize>true</visualize>
+      <imu>
+        <!-- Gyroscope noise (angular velocity in rad/s) -->
+        <angular_velocity>
+          <x>
+            <noise type="gaussian">
+              <mean>0.0</mean>
+              <stddev>${noise}</stddev>        <!-- noise strength -->
+              <bias_mean>0.0</bias_mean>
+              <bias_stddev>${drift}</bias_stddev> <!-- slow drift -->
+            </noise>
+          </x>
+          <y>
+            <noise type="gaussian">
+              <mean>0.0</mean>
+              <stddev>${noise}</stddev>
+              <bias_mean>0.0</bias_mean>
+              <bias_stddev>${drift}</bias_stddev>
+            </noise>
+          </y>
+          <z>
+            <noise type="gaussian">
+              <mean>0.0</mean>
+              <stddev>${noise}</stddev>
+              <bias_mean>0.0</bias_mean>
+              <bias_stddev>${drift}</bias_stddev>
+            </noise>
+          </z>
+        </angular_velocity>
+        <!-- Accelerometer noise (linear acceleration in m/s^2) -->
+        <linear_acceleration>
+          <x>
+            <noise type="gaussian">
+              <mean>0.0</mean>
+              <stddev>${noise}</stddev>         <!-- higher noise -->
+              <bias_mean>0.0</bias_mean>
+              <bias_stddev>${drift}</bias_stddev>
+            </noise>
+          </x>
+          <y>
+            <noise type="gaussian">
+              <mean>0.0</mean>
+              <stddev>${noise}</stddev>
+              <bias_mean>0.0</bias_mean>
+              <bias_stddev>${drift}</bias_stddev>
+            </noise>
+          </y>
+          <z>
+            <noise type="gaussian">
+              <mean>0.0</mean>
+              <stddev>${noise}</stddev>
+              <bias_mean>0.0</bias_mean>
+              <bias_stddev>${drift}</bias_stddev>
+            </noise>
+          </z>
+        </linear_acceleration>
+      </imu>
+      <!-- ROS plugin to publish /imu -->
       <plugin name="imu_plugin" filename="libgazebo_ros_imu_sensor.so">
         <ros>

Commit message: added realistic noise and drift to IMU sensor. Close approximation to model_states

File: src/latty_chassis/urdf/latty_model.urdf.xacro (robot description, xacro)
@@ -261,5 +261,5 @@
     </joint>
   </ros2_control>
-  <xacro:property name="noise" value="1e-3"/>
+  <xacro:property name="noise" value="0.1"/>
   <xacro:property name="drift" value="1e-5"/>
   <gazebo>
@@ -273,4 +273,60 @@
       <update_rate>100.0</update_rate>   <!-- 100 Hz IMU -->
       <visualize>true</visualize>
+      <imu>
+        <!-- Gyroscope noise (angular velocity in rad/s) -->
+        <angular_velocity>
+          <x>
+            <noise type="gaussian">
+              <mean>0.0</mean>
+              <stddev>${noise}</stddev>        <!-- noise strength -->
+              <bias_mean>0.0</bias_mean>
+              <bias_stddev>${drift}</bias_stddev> <!-- slow drift -->
+            </noise>
+          </x>
+          <y>
+            <noise type="gaussian">
+              <mean>0.0</mean>
+              <stddev>${noise}</stddev>
+              <bias_mean>0.0</bias_mean>
+              <bias_stddev>${drift}</bias_stddev>
+            </noise>
+          </y>
+          <z>
+            <noise type="gaussian">
+              <mean>0.0</mean>
+              <stddev>${noise}</stddev>
+              <bias_mean>0.0</bias_mean>
+              <bias_stddev>${drift}</bias_stddev>
+            </noise>
+          </z>
+        </angular_velocity>
+        <!-- Accelerometer noise (linear acceleration in m/s^2) -->
+        <linear_acceleration>
+          <x>
+            <noise type="gaussian">
+              <mean>0.0</mean>
+              <stddev>${noise}</stddev>         <!-- higher noise -->
+              <bias_mean>0.0</bias_mean>
+              <bias_stddev>${drift}</bias_stddev>
+            </noise>
+          </x>
+          <y>
+            <noise type="gaussian">
+              <mean>0.0</mean>
+              <stddev>${noise}</stddev>
+              <bias_mean>0.0</bias_mean>
+              <bias_stddev>${drift}</bias_stddev>
+            </noise>
+          </y>
+          <z>
+            <noise type="gaussian">
+              <mean>0.0</mean>
+              <stddev>${noise}</stddev>
+              <bias_mean>0.0</bias_mean>
+              <bias_stddev>${drift}</bias_stddev>
+            </noise>
+          </z>
+        </linear_acceleration>
+      </imu>
       <!-- ROS plugin to publish /imu -->
       <plugin name="imu_plugin" filename="libgazebo_ros_imu_sensor.so">

Commit message: added more dynamic vehicle model with differential drive during sharp turns

File: src/latty_chassis/urdf/latty_model.urdf.xacro (robot description, xacro)
@@ -4,5 +4,5 @@
   <xacro:property name="wheel_radius" value="0.1"/>
   <xacro:property name="wheel_length" value="0.06"/>
-  <xacro:property name="front_wheel_radius" value="0.03"/>
+  <xacro:property name="front_wheel_radius" value="0.02"/>
   <xacro:property name="front_wheel_length" value="0.02"/>
   <xacro:property name="wheelbase" value="0.25"/>
@@ -132,5 +132,5 @@
     </collision>
     <inertial>
-      <origin xyz="0 0 0"  rpy="0 0 0"/>
+      <origin xyz="0 0 0" rpy="0 0 0"/>
       <mass value="0.01"/>
       <inertia ixx="1e-6" iyy="1e-6" izz="1e-6" ixy="0" ixz="0" iyz="0"/>
@@ -147,16 +147,24 @@
     <material>Gazebo/Yellow</material>
   </gazebo>
+  <xacro:property name="frontWheel_mu1" value="0.5"/>
+  <xacro:property name="frontWheel_mu2" value="0.1"/>
+  <xacro:property name="rearWheel_mu1" value="1.0"/>
+  <xacro:property name="rearWheel_mu2" value="0.5"/>
+  <xacro:property name="fdir1_q" value="0 0 1"/>
   <gazebo reference="left_wheel">
     <material>Gazebo/Black</material>
-    <mu1>1.0</mu1>
-    <mu2>1.0</mu2>
-    <kp>1000000.0</kp>
+    <!-- make lateral (mu1) big, longitudinal (mu2) moderate -->
+    <fdir1>${fdir1_q}</fdir1>
+    <mu1>${rearWheel_mu1}</mu1>    <!-- lateral -->
+    <mu2>${rearWheel_mu2}</mu2>    <!-- longitudinal -->
+    <kp>1e6</kp>
     <kd>1.0</kd>
   </gazebo>
   <gazebo reference="right_wheel">
     <material>Gazebo/Black</material>
-    <mu1>1.0</mu1>
-    <mu2>1.0</mu2>
-    <kp>1000000.0</kp>
+    <fdir1>${fdir1_q}</fdir1>
+    <mu1>${rearWheel_mu1}</mu1>    <!-- lateral -->
+    <mu2>${rearWheel_mu2}</mu2>    <!-- longitudinal -->
+    <kp>1e6</kp>
     <kd>1.0</kd>
   </gazebo>
@@ -168,14 +176,16 @@
   <gazebo reference="front_left_wheel">
     <material>Gazebo/Black</material>
-    <mu1>1.0</mu1>
-    <mu2>1.0</mu2>
-    <kp>1000000.0</kp>
+    <fdir1>${fdir1_q}</fdir1>
+    <mu1>${frontWheel_mu1}</mu1>    <!-- lateral -->
+    <mu2>${frontWheel_mu2}</mu2>    <!-- longitudinal -->
+    <kp>1e6</kp>
     <kd>1.0</kd>
   </gazebo>
   <gazebo reference="front_right_wheel">
     <material>Gazebo/Black</material>
-    <mu1>1.0</mu1>
-    <mu2>1.0</mu2>
-    <kp>1000000.0</kp>
+    <fdir1>${fdir1_q}</fdir1>
+    <mu1>${frontWheel_mu1}</mu1>    <!-- lateral -->
+    <mu2>${frontWheel_mu2}</mu2>    <!-- longitudinal -->
+    <kp>1e6</kp>
     <kd>1.0</kd>
   </gazebo>
@@ -200,5 +210,5 @@
     <origin xyz="-0.15 0 0.03" rpy="0 0 0"/>
     <axis xyz="0 0 1"/>
-    <limit lower="-0.785" upper="0.785" effort="10" velocity="3"/>
+    <limit lower="-0.5236" upper="0.5236" effort="10" velocity="3"/>
     <dynamics damping="0.5"/>
   </joint>
@@ -207,5 +217,5 @@
     <parent link="steer_knuckle"/>
     <child link="front_left_wheel"/>
-    <origin xyz="0 0.02 -0.015" rpy="0 0 0"/>
+    <origin xyz="0 0.02 -0.01" rpy="0 0 0"/>
     <axis xyz="0 -1 0"/>
     <dynamics damping="0.1" friction="0.05"/>
@@ -214,5 +224,5 @@
     <parent link="steer_knuckle"/>
     <child link="front_right_wheel"/>
-    <origin xyz="0 -0.02 -0.015" rpy="0 0 0"/>
+    <origin xyz="0 -0.02 -0.01" rpy="0 0 0"/>
     <axis xyz="0 -1 0"/>
     <dynamics damping="0.1" friction="0.05"/>
@@ -222,5 +232,5 @@
     <parent link="chassis"/>
     <child link="left_wheel"/>
-    <origin xyz="0.1 0.13 0.085" rpy="0 0 0"/>
+    <origin xyz="0.1 0.13 ${wheel_radius}" rpy="0 0 0"/>
     <axis xyz="0 -1 0"/>
     <dynamics damping="5.0" friction="0.5"/>
@@ -229,5 +239,5 @@
     <parent link="chassis"/>
     <child link="right_wheel"/>
-    <origin xyz="0.1 -0.13 0.085" rpy="0 0 0"/>
+    <origin xyz="0.1 -0.13 ${wheel_radius}" rpy="0 0 0"/>
     <axis xyz="0 -1 0"/>
     <dynamics damping="5.0" friction="0.5"/>
@@ -261,6 +271,6 @@
     </joint>
   </ros2_control>
-  <xacro:property name="noise" value="0.1"/>
-  <xacro:property name="drift" value="1e-5"/>
+  <xacro:property name="noise" value="0.005"/>
+  <xacro:property name="drift" value="1e-6"/>
   <gazebo>
     <plugin name="gazebo_ros2_control" filename="libgazebo_ros2_control.so">
@@ -271,5 +281,5 @@
     <sensor name="imu_sensor" type="imu">
       <always_on>true</always_on>
-      <update_rate>100.0</update_rate>   <!-- 100 Hz IMU -->
+      <update_rate>100.0</update_rate>      <!-- 100 Hz IMU -->
       <visualize>true</visualize>
       <imu>
@@ -279,7 +289,7 @@
             <noise type="gaussian">
               <mean>0.0</mean>
-              <stddev>${noise}</stddev>        <!-- noise strength -->
-              <bias_mean>0.0</bias_mean>
-              <bias_stddev>${drift}</bias_stddev> <!-- slow drift -->
+              <stddev>${noise}</stddev>              <!-- noise strength -->
+              <bias_mean>0.0</bias_mean>
+              <bias_stddev>${drift}</bias_stddev>              <!-- slow drift -->
             </noise>
           </x>
@@ -306,5 +316,5 @@
             <noise type="gaussian">
               <mean>0.0</mean>
-              <stddev>${noise}</stddev>         <!-- higher noise -->
+              <stddev>${noise}</stddev>              <!-- higher noise -->
               <bias_mean>0.0</bias_mean>
               <bias_stddev>${drift}</bias_stddev>
