Commit message: lidar added, as well as a cafe setup environment in gazebo to map

File: src/latty_chassis/urdf/latty_model.urdf.xacro (robot description, xacro)
@@ -7,4 +7,6 @@
   <xacro:property name="front_wheel_length" value="0.02"/>
   <xacro:property name="wheelbase" value="0.25"/>
+  <xacro:property name="lidar_radius" value="0.05"/>
+  <xacro:property name="lidar_length" value="0.1"/>
   <link name="base_link"/>
   <!-- Chassis -->
@@ -134,5 +136,7 @@
       <origin xyz="0 0 0" rpy="0 0 0"/>
       <mass value="0.01"/>
-      <inertia ixx="1e-6" iyy="1e-6" izz="1e-6" ixy="0" ixz="0" iyz="0"/>
+      <inertia
+        ixx="2.4e-05" iyy="2.4e-05" izz="4.2e-05"
+        ixy="0.0" ixz="0.0" iyz="0.0"/>
     </inertial>
     <visual>
@@ -140,4 +144,26 @@
       <geometry>
         <box size="0.05 0.05 0.02"/>
+      </geometry>
+    </visual>
+  </link>
+  <!-- Lidar Link -->
+  <link name="lidar_link">
+    <collision>
+      <origin xyz="0 0 0" rpy="0 0 0"/>
+      <geometry>
+        <cylinder length="${lidar_length}" radius="${lidar_radius}"/>
+      </geometry>
+    </collision>
+    <inertial>
+      <origin xyz="0 0 0" rpy="0 0 0"/>
+      <mass value="0.01"/>
+      <inertia
+        ixx="2.2e-05" iyy="2.2e-05" izz="4.5e-06"
+        ixy="0.0" ixz="0.0" iyz="0.0"/>
+    </inertial>
+    <visual>
+      <origin xyz="0 0 0" rpy="0 0 0"/>
+      <geometry>
+        <cylinder length="${lidar_length}" radius="${lidar_radius}"/>
       </geometry>
     </visual>
@@ -193,4 +219,7 @@
     <material>Gazebo/Grey</material>
   </gazebo>
+  <gazebo reference="lidar_link">
+    <material>Gazebo/Blue</material>
+  </gazebo>
   <!-- Joints -->
   <joint name="base_to_chassis" type="fixed">
@@ -203,5 +232,10 @@
     <parent link="base_link"/>
     <child link="imu_link"/>
-    <origin xyz="-0.05 0 0.16" rpy="0 0 0"/>
+    <origin xyz="-0.1 0 0.16" rpy="0 0 0"/>
+  </joint>
+  <joint name="lidar_joint" type="fixed">
+    <parent link="base_link"/>
+    <child link="lidar_link"/>
+    <origin xyz="0.1 0 0.16" rpy="0 0 0"/>
   </joint>
   <joint name="front_steer_joint" type="revolute">
@@ -349,3 +383,39 @@
     </sensor>
   </gazebo>
+  <gazebo reference="lidar_link">
+    <sensor name="laser" type="ray">
+      <pose>0 0 0 0 0 0</pose>
+      <always_on>true</always_on>
+      <visualize>true</visualize>
+      <update_rate>100</update_rate>
+      <ray>
+        <scan>
+          <horizontal>
+            <samples>360</samples>
+            <resolution>1</resolution>
+            <min_angle>-3.14</min_angle>
+            <max_angle>3.14</max_angle>
+          </horizontal>
+        </scan>
+        <range>
+          <min>0.3</min>
+          <max>12.0</max>
+          <resolution>0.01</resolution>
+        </range>
+        <noise>
+          <type>gaussian</type>
+          <mean>0.0</mean>
+          <stddev>0.01</stddev>
+        </noise>
+      </ray>
+      <plugin name="gazebo_ros_laser" filename="libgazebo_ros_ray_sensor.so">
+        <ros>
+          <namespace>/</namespace>
+          <remapping>~/out:=/scan</remapping>
+        </ros>
+        <output_type>sensor_msgs/LaserScan</output_type>
+        <frame_name>lidar_link</frame_name>
+      </plugin>
+    </sensor>
+  </gazebo>
 </robot>
